File: Checkpoint 2/kicad/Proyecto Integrador G1.kicad_sch (KiCad schematic)
At the start: 50 parts, among them J1 Conn_01x02, J2 Conn_01x02, Q1 BC547, Q10 BC547, Q2 BC547, Q3 BC547, Q4 BC547, Q5 BC557, Q6 BC557, Q7 BC547, Q8 TIP42C, Q9 BC547, U1 TL431LP, U2 LM358

Commit message: rev 1.1
Other:
- moved on the sheet: C1, C_c1, J1, J2, JP_FES1, JP_VL1, JP_VL2, JP_comp1, JP_reg1, Q1, Q10, Q2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

Commit message: rev 1.2
Parts:
- added R2_2, R2p_2, R3_2, R3p_2: 1M, Resistor_THT:R_Axial_DIN0207_L6.3mm_D2.5mm_P7.62mm_Horizontal, symbol Device:R
- C1: value 100nF -> 100n
- C_c1: value 100n -> 1u
- Q8: value TIP42C -> TIP32C
- R2_1: renamed from R2; value 500k -> 1M
- R2p_1: renamed from R2p1; value 500k -> 1M
- R3_1: renamed from R3; value 500k -> 1M
- R3p_1: renamed from R3p1; value 500k -> 1M
- R_ref1: value 3k3 -> 1k
Connections:
- net GND: now also JP_comp1.2 (B), R2p_2.1, R3p_2.1
- net Vb: now also R_c1.1; no longer JP_comp1.1 (A)
- net Vout: now also R3_2.1
- net Vref: no longer R_c1.1, R_ref1.2
- net Vreg: now also R_ref1.2, R2_2.1
- net at R1p1.2, R2p_1.2, R3p_1.2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: now also R2p_2.2, R3p_2.2
- net at R1.2, R2_1.2, R3_1.2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: now also R2_2.2, R3_2.2
- net at C_c1.2: now also JP_comp1.1 (A); no longer JP_comp1.2 (B)
Other:
- moved on the sheet: R2p_1, R3_1, R3p_1
